File: Hardware/MotherBoard/BusExtentions.kicad_sch (KiCad schematic)
At the start: 10 parts, among them J3 ISA00, J4 ISA10, J7 ISA01, J8 ISA11, U10 SN74LVC245AN, U11 SN74LVC245AN, U12 SN74LVC245AN, U13 74HCT541, U14 74HCT541, U9 SN74LVC245AN

Commit message: Version 1.2
Parts:
- U10, U11, U12, U9: value SN74LVC245AN -> 74HC245; Category Integrated Circuits (ICs) -> (none); DK_Datasheet_Link http://www.ti.com/general/docs/suppproductinfo.tsp?distId=1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 -> (none); DK_Detail_Page /product-detail/en/texas-instruments/SN74LVC245AN/296-8503-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 -> (none); Digi-Key_PN 296-8503-5-ND -> (none); Family Logic - Buffers, Drivers, Receivers, Transceivers -> (none); MPN SN74LVC245AN -> (none); Manufacturer Texas Instruments -> (none); Status Active -> (none)
- U13, U14: value 74HCT541 -> 74HC541
Connections:
- net +5V: now also J3.16 (Pin_16), J4.16 (Pin_16); no longer J3.15 (Pin_15), J4.15 (Pin_15)
- net A0: now also U9.2 (A1); no longer U9.18 (B1)
- net A1: now also U9.3 (A2); no longer U9.17 (B2)
- net A10: now also U10.4 (A3); no longer U10.16 (B3)
- net A11: now also U10.5 (A4); no longer U10.15 (B4)
- net A12: now also U10.6 (A5); no longer U10.14 (B5)
- net A13: now also U10.7 (A6); no longer U10.13 (B6)
- net A14: now also U10.8 (A7); no longer U10.12 (B7)
- net A2: now also U9.4 (A3); no longer U9.16 (B3)
- net A3: now also U9.5 (A4); no longer U9.15 (B4)
- net A4: now also U9.6 (A5); no longer U9.14 (B5)
- net A5: now also U9.7 (A6); no longer U9.13 (B6)
- net A6: now also U9.8 (A7); no longer U9.12 (B7)
- net A7: now also U9.9 (A8); no longer U9.11 (B8)
- net A8: now also U10.2 (A1); no longer U10.18 (B1)
- net A9: now also U10.3 (A2); no longer U10.17 (B2)
- net GND: now also J3.15 (Pin_15); no longer J7.16 (Pin_16), J8.16 (Pin_16), U13.9 (A7)
- net RDYB: now also J4.15 (Pin_15); no longer J4.16 (Pin_16)
- net at J8.1 (Pin_1): now also U9.18 (B1); no longer U9.2 (A1)
- net at J8.10 (Pin_10): now also U10.17 (B2); no longer U10.3 (A2)
- net at J8.11 (Pin_11): now also U10.16 (B3); no longer U10.4 (A3)
- net at J8.12 (Pin_12): now also U10.15 (B4); no longer U10.5 (A4)
- net at J8.13 (Pin_13): now also U10.14 (B5); no longer U10.6 (A5)
- net at J8.14 (Pin_14): now also U10.13 (B6); no longer U10.7 (A6)
- net at J8.15 (Pin_15): now also U10.12 (B7); no longer U10.8 (A7)
- net at J8.2 (Pin_2): now also U9.17 (B2); no longer U9.3 (A2)
- net at J8.3 (Pin_3): now also U9.16 (B3); no longer U9.4 (A3)
- net at J8.4 (Pin_4): now also U9.15 (B4); no longer U9.5 (A4)
- net at J8.5 (Pin_5): now also U9.14 (B5); no longer U9.6 (A5)
- net at J8.6 (Pin_6): now also U9.13 (B6); no longer U9.7 (A6)
- net at J8.7 (Pin_7): now also U9.12 (B7); no longer U9.8 (A7)
- net at J8.8 (Pin_8): now also U9.11 (B8); no longer U9.9 (A8)
- net at J8.9 (Pin_9): now also U10.18 (B1); no longer U10.2 (A1)
- net at U13.11 (Y7): now also J7.16 (Pin_16)
- net IRQ0B: now reaches J3.11 (Pin_11)
- net at U10.11 (B8): now also J8.16 (Pin_16)
- net A15: now reaches U10.9 (A8)
- net A15: now also U13.9 (A7)
- no-connect marks 5 -> 0
Other:
- moved on the sheet: U10, U9
