File: Hardware/AdapterCartdrige/AdapterCartdrige.kicad_sch (KiCad schematic)
At the start: 3 parts, among them J1 ROM, U1 28C256

Commit message: Fix
Connections:
- no-connect marks 0 -> 2
Other:
- moved on the sheet: C1
