File: Hardware/AdapterCartdrigeProd/AdapterCartdrigeProd.kicad_sch (KiCad schematic)
At the start: 5 parts, among them J1 ROM, U1 28C256

Commit message: Fix
Parts:
- added H3: MountingHole_Pad, MountingHole:MountingHole_3.2mm_M3, symbol Mechanical:MountingHole_Pad
Connections:
- net GND: now also H3.1
Other:
- moved on the sheet: C1, J1, U1
