File: Hardware/Cartdrige/Cartdrige.kicad_pcb (KiCad board)
At the start: 2 copper layers, 80 x 34.3 mm, 4 parts, among them J1 ROM, U1 28C256

Commit message: Finalize 1.3
Parts:
- removed J1: ROM, Connector_TheRLab:NES_PCBEdge
- removed the XiaoNiuNiu at (87.9, 32.0)
- added J2: PORT1, NESConnector:NES_PCBEdge, F.Cu at (110.5, 91.7)
- added XiaoNiuNiu: LOGO, Cow:VerySmallCow, F.Cu at (81.0, 81.0)
- moved C1 64.5 mm to (136.1, 76.9), turned to 90 degrees
- moved U1 58.8 mm to (128.3, 61.7)
Connections:
- U1 pad 20: CS -> /PORT1CSB
- U1 pad 22: OE -> /CLOCK
Routing:
- net +5V: track 83.3 -> 180.4 mm, vias 2 -> 1
- net /CLOCK: track 0.00 -> 56.0 mm, vias 0 -> 1
- net OE: track 55.1 -> 0.00 mm
- net /A7: track 47.7 -> 100.3 mm, vias 0 -> 1
- net CS: track 50.5 -> 0.00 mm
- net /A6: track 48.6 -> 89.9 mm, vias 0 -> 1
- net /A5: track 49.5 -> 79.6 mm, vias 0 -> 1
- net /D3: track 32.9 -> 55.6 mm, vias 0 -> 1
- net /A13: track 52.1 -> 31.6 mm, vias 0 -> 1
- net /A4: track 50.4 -> 69.2 mm, vias 0 -> 1
- net /PORT1CSB: track 0.00 -> 17.6 mm
- net GND: track 16.0 -> 0.00 mm, vias 3 -> 0
- net /D4: track 38.6 -> 54.5 mm, vias 0 -> 1
- net /A8: track 48.8 -> 36.1 mm, vias 0 -> 2
- net /D5: track 41.3 -> 53.4 mm, vias 0 -> 1
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Other:
- board text added: "+"

Commit message: Version 1.3
Parts:
- moved C1 9.78 mm to (145.9, 77.0)
Connections:
- U1 pad 22: /CLOCK -> GND
Routing:
- net /CLOCK: track 56.0 -> 0.00 mm, vias 1 -> 0
- net +5V: track 180.4 -> 192.9 mm
- net /A9: track 44.0 -> 43.0 mm
- net /A8: track 36.1 -> 35.5 mm
Changed lines of the file:
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@@
   (net 58 "unconnected-(J2-Pin_60-Pad60)")
   (footprint "Capacitor_THT:C_Disc_D5.0mm_W2.5mm_P2.50mm" (layer "F.Cu")
-    (at 136.144 76.942 90)
+    (at 145.923 76.962 90)
     (descr "C, Disc series, Radial, pin pitch=2.50mm, , diameter*width=5*2.5mm^2, Capacitor, http://cdn-reichelt.de/documents/datenblatt/B300/DS_KERKO_TC.pdf")
     (tags "C Disc series Radial pin pitch 2.50mm  diameter 5mm width 2.5mm Capacitor")
@@
     (property "ki_keywords" "Parallel EEPROM 256Kb")
     (attr through_hole)
-    (fp_text reference "U1" (at 7.62 -2.33 -90) (layer "F.SilkS")
+    (fp_text reference "U1" (at 7.62 16.51 -90) (layer "F.SilkS")
         (effects (font (size 1 1) (thickness 0.15)))
     )
@@
       (net 7 "/A10") (pinfunction "A10") (pintype "input"))
     (pad "22" thru_hole oval (at 15.24 15.24 270) (size 1.6 1.6) (drill 0.8) (layers "*.Cu" "*.Mask")
-      (net 26 "/CLOCK") (pinfunction "~{OE}") (pintype "input"))
+      (net 1 "GND") (pinfunction "~{OE}") (pintype "input"))
     (pad "23" thru_hole oval (at 15.24 12.7 270) (size 1.6 1.6) (drill 0.8) (layers "*.Cu" "*.Mask")
       (net 6 "/A11") (pinfunction "A11") (pintype "input"))
@@
     (effects (font (size 1 1) (thickness 0.15)) (justify left bottom))
   )
+  (segment (start 145.923 76.962) (end 148.463 76.962) (width 0.5) (layer "F.Cu") (net 2))
+  (segment (start 148.463 76.962) (end 148.59 76.835) (width 0.5) (layer "F.Cu") (net 2))
   (segment (start 148.59 57.15) (end 145.288 53.848) (width 0.5) (layer "F.Cu") (net 2))
   (segment (start 128.27 76.962) (end 128.27 67.056) (width 0.5) (layer "F.Cu") (net 2))
   (segment (start 74.93 57.658) (end 74.93 86.106) (width 0.5) (layer "F.Cu") (net 2))
+  (segment (start 148.59 91.694) (end 148.59 76.835) (width 0.5) (layer "F.Cu") (net 2))
   (segment (start 132.334 53.848) (end 78.74 53.848) (width 0.5) (layer "F.Cu") (net 2))
-  (segment (start 148.59 91.694) (end 148.59 57.15) (width 0.5) (layer "F.Cu") (net 2))
   (segment (start 132.334 62.992) (end 132.334 53.848) (width 0.5) (layer "F.Cu") (net 2))
+  (segment (start 148.59 76.835) (end 148.59 57.15) (width 0.5) (layer "F.Cu") (net 2))
   (segment (start 145.288 53.848) (end 132.334 53.848) (width 0.5) (layer "F.Cu") (net 2))
   (segment (start 78.74 53.848) (end 74.93 57.658) (width 0.5) (layer "F.Cu") (net 2))
@@
   (segment (start 74.93 91.694) (end 74.93 86.106) (width 0.5) (layer "B.Cu") (net 2))
   (segment (start 125.73 76.962) (end 128.27 76.962) (width 0.5) (layer "B.Cu") (net 2))
-  (segment (start 128.27 76.962) (end 136.144 76.942) (width 0.5) (layer "B.Cu") (net 2))
+  (segment (start 128.27 76.962) (end 145.923 76.962) (width 0.5) (layer "B.Cu") (net 2))
   (segment (start 140.97 91.694) (end 140.97 78.486) (width 0.3) (layer "F.Cu") (net 3))
   (via (at 140.97 78.486) (size 0.8) (drill 0.4) (layers "F.Cu" "B.Cu") (net 3))
   (segment (start 123.19 76.962) (end 124.714 78.486) (width 0.3) (layer "B.Cu") (net 3))
   (segment (start 124.714 78.486) (end 140.97 78.486) (width 0.3) (layer "B.Cu") (net 3))
-  (segment (start 134.112 83.058) (end 134.112 81.026) (width 0.3) (layer "F.Cu") (net 4))
-  (segment (start 134.112 81.026) (end 134.112 72.644) (width 0.3) (layer "F.Cu") (net 4))
-  (via (at 134.112 83.058) (size 0.8) (drill 0.4) (layers "F.Cu" "B.Cu") (net 4))
-  (via (at 134.112 72.644) (size 0.8) (drill 0.4) (layers "F.Cu" "B.Cu") (net 4))
+  (segment (start 137.414 74.422) (end 137.414 77.724) (width 0.3) (layer "F.Cu") (net 4))
+  (segment (start 137.414 77.724) (end 137.414 86.36) (width 0.3) (layer "F.Cu") (net 4))
+  (via (at 137.414 74.422) (size 0.8) (drill 0.4) (layers "F.Cu" "B.Cu") (net 4))
+  (via (at 137.414 86.36) (size 0.8) (drill 0.4) (layers "F.Cu" "B.Cu") (net 4))
+  (segment (start 137.414 86.36) (end 138.43 87.376) (width 0.3) (layer "B.Cu") (net 4))
+  (segment (start 137.414 74.422) (end 123.19 74.422) (width 0.3) (layer "B.Cu") (net 4))
+  (segment (start 123.19 74.422) (end 120.65 76.962) (width 0.3) (layer "B.Cu") (net 4))
   (segment (start 138.43 87.376) (end 138.43 91.694) (width 0.3) (layer "B.Cu") (net 4))
-  (segment (start 134.112 83.058) (end 138.43 87.376) (width 0.3) (layer "B.Cu") (net 4))
-  (segment (start 124.968 72.644) (end 120.65 76.962) (width 0.3) (layer "B.Cu") (net 4))
-  (segment (start 134.112 72.644) (end 124.968 72.644) (width 0.3) (layer "B.Cu") (net 4))
-  (segment (start 139.7 71.882) (end 139.7 86.36) (width 0.3) (layer "F.Cu") (net 5))
+  (segment (start 139.7 72.644) (end 139.7 86.36) (width 0.3) (layer "F.Cu") (net 5))
   (via (at 139.7 86.36) (size 0.8) (drill 0.4) (layers "F.Cu" "B.Cu") (net 5))
-  (via (at 139.7 71.882) (size 0.8) (drill 0.4) (layers "F.Cu" "B.Cu") (net 5))
+  (via (at 139.7 72.644) (size 0.8) (drill 0.4) (layers "F.Cu" "B.Cu") (net 5))
+  (segment (start 139.7 72.644) (end 122.428 72.644) (width 0.3) (layer "B.Cu") (net 5))
+  (segment (start 122.428 72.644) (end 118.11 76.962) (width 0.3) (layer "B.Cu") (net 5))
   (segment (start 140.97 87.63) (end 140.97 91.694) (width 0.3) (layer "B.Cu") (net 5))
-  (segment (start 139.7 71.882) (end 123.19 71.882) (width 0.3) (layer "B.Cu") (net 5))
   (segment (start 139.7 86.36) (end 140.97 87.63) (width 0.3) (layer "B.Cu") (net 5))
-  (segment (start 123.19 71.882) (end 118.11 76.962) (width 0.3) (layer "B.Cu") (net 5))
   (segment (start 137.668 79.248) (end 117.856 79.248) (width 0.3) (layer "B.Cu") (net 6))
   (segment (start 146.05 91.694) (end 146.05 87.63) (width 0.3) (layer "B.Cu") (net 6))
@@
   (segment (start 109.22 83.312) (end 111.252 85.344) (width 0.3) (layer "B.Cu") (net 17))
   (segment (start 120.65 87.63) (end 120.65 91.694) (width 0.3) (layer "B.Cu") (net 17))
-  (segment (start 111.252 85.344) (end 111.76 85.344) (width 0.3) (layer "B.Cu") (net 17))
-  (segment (start 111.76 85.344) (end 118.364 85.344) (width 0.3) (layer "B.Cu") (net 17))
+  (segment (start 111.252 85.344) (end 118.364 85.344) (width 0.3) (layer "B.Cu") (net 17))
   (segment (start 111.76 62.992) (end 110.49 61.722) (width 0.3) (layer "F.Cu") (net 18))
   (segment (start 111.76 84.582) (end 111.76 62.992) (width 0.3) (layer "F.Cu") (net 18))
@@
   (segment (start 138.303 61.722) (end 138.43 61.595) (width 0.3) (layer "B.Cu") (net 25))
   (segment (start 128.27 61.722) (end 138.303 61.722) (width 0.3) (layer "B.Cu") (net 25))
-  (segment (start 146.05 71.12) (end 146.05 91.694) (width 0.3) (layer "F.Cu") (net 26))
-  (via (at 146.05 71.12) (size 0.8) (drill 0.4) (layers "F.Cu" "B.Cu") (net 26))
-  (segment (start 118.872 71.12) (end 113.03 76.962) (width 0.3) (layer "B.Cu") (net 26))
-  (segment (start 146.05 71.12) (end 118.872 71.12) (width 0.3) (layer "B.Cu") (net 26))
   (segment (start 110.49 86.36) (end 107.95 83.82) (width 0.3) (layer "F.Cu") (net 30))
   (segment (start 113.03 87.63) (end 111.76 86.36) (width 0.3) (layer "F.Cu") (net 30))

Commit message: A lot of new hardware
Parts:
- J2: footprint NESConnector:NES_PCBEdge -> Connector_NES:NES_PCBEdge
- moved XiaoNiuNiu 0.57 mm to (81.3, 80.5)
Changed lines of the file:
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@@
   )
   (footprint "Cow:VerySmallCow" (layer "F.Cu")
-    (at 81.026 81.026)
+    (at 81.28 80.518)
     (attr through_hole)
     (fp_text reference "XiaoNiuNiu" (at 9.906 3.81) (layer "F.SilkS")
@@
       (stroke (width 0) (type solid)) (fill solid) (layer "F.SilkS"))
   )
-  (footprint "NESConnector:NES_PCBEdge" (layer "F.Cu")
+  (footprint "Connector_NES:NES_PCBEdge" (layer "F.Cu")
     (at 110.49 91.694)
     (descr "NES Cartdrige Edge Connector")
