File: Hardware/CartdrigeDev/CartdrigeDev.kicad_sch (KiCad schematic)
At the start: 2 parts, among them J1 Conn_02x30_Odd_Even, J2 PORT1

Commit message: Version 1.3
Parts:
- removed J1: Conn_02x30_Odd_Even, Connector_PinSocket_2.54mm:PinSocket_2x30_P2.54mm_Vertical, symbol Connector_Generic:Conn_02x30_Odd_Even
- added C1: 100nF, Capacitor_THT:C_Disc_D5.0mm_W2.5mm_P2.50mm, symbol Device:C
- added U1: 28C256, Socket:DIP_Socket-28_W11.9_W12.7_W15.24_W17.78_W18.5_3M_228-1277-00-0602J, symbol Memory_EEPROM:28C256
Connections:
- net +5V: now also C1.1, U1.27 (~{WE}), U1.28 (VCC)
- net A0: now also U1.10 (A0)
- net A1: now also U1.9 (A1)
- net A10: now also U1.21 (A10)
- net A11: now also U1.23 (A11)
- net A12: now also U1.2 (A12)
- net A13: now also U1.26 (A13)
- net A14: now also U1.1 (A14)
- net A2: now also U1.8 (A2)
- net A3: now also U1.7 (A3)
- net A4: now also U1.6 (A4)
- net A5: now also U1.5 (A5)
- net A6: now also U1.4 (A6)
- net A7: now also U1.3 (A7)
- net A8: now also U1.25 (A8)
- net A9: now also U1.24 (A9)
- net D0: now also U1.11 (D0)
- net D1: now also U1.12 (D1)
- net D2: now also U1.13 (D2)
- net D3: now also U1.15 (D3)
- net D4: now also U1.16 (D4)
- net D5: now also U1.17 (D5)
- net D6: now also U1.18 (D6)
- net D7: now also U1.19 (D7)
- net GND: now also C1.2, U1.14 (GND), U1.22 (~{OE})
- net PORT1CSB: now also U1.20 (~{CS})
- no-connect marks 48 -> 24

Commit message: A lot of new hardware
Parts:
- J2: footprint NESConnector:NES_PCBEdge -> Connector_NES:NES_PCBEdge
- U1: footprint Socket:DIP_Socket-28_W11.9_W12.7_W15.24_W17.78_W18.5_3M_228-1277-00-0602J -> Package_DIP:DIP-28_W7.62mm
Connections:
- net A15: no longer names the net of J2.12 (Pin_12)
- net CLOCK: no longer names the net of J2.4 (Pin_4)
- net DMAB: no longer names the net of J2.34 (Pin_34)
- net IRQ3B: no longer names the net of J2.29 (Pin_29)
- net NMIB: no longer names the net of J2.36 (Pin_36)
- net RAMCSB: no longer names the net of J2.33 (Pin_33)
- net RESET: no longer names the net of J2.32 (Pin_32)
- net RW: no longer names the net of J2.27 (Pin_27)
- no-connect marks 24 -> 32
Other:
- moved on the sheet: C1
