File: Hardware/CartdrigeProto/CartdrigeProto.kicad_pcb (KiCad board)
At the start: 2 copper layers, 80 x 14.5 mm, 2 parts, among them J1 Conn_02x30_Odd_Even, J2 PORT1

Commit message: A lot of new hardware
Parts:
- J2: footprint NESConnector:NES_PCBEdge -> Connector_NES:NES_PCBEdge
Changed lines of the file:
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@@
   (net 81 "unconnected-(J1-Pin_58-Pad58)")
   (net 82 "unconnected-(J1-Pin_60-Pad60)")
-  (footprint "NESConnector:NES_PCBEdge" (layer "F.Cu")
+  (footprint "Connector_NES:NES_PCBEdge" (layer "F.Cu")
     (at 110.49 91.694)
     (descr "NES Cartdrige Edge Connector")
     (tags "NES Edge connector")
-    (property "Sheetfile" "CartdrigeDev.kicad_sch")
+    (property "Sheetfile" "CartdrigeProto.kicad_sch")
     (property "Sheetname" "")
     (property "ki_description" "Generic connector, double row, 02x30, odd/even pin numbering scheme (row 1 odd numbers, row 2 even numbers), script generated (kicad-library-utils/schlib/autogen/connector/)")
@@
     (descr "Through hole straight socket strip, 2x30, 2.54mm pitch, double cols (from Kicad 4.0.7), script generated")
     (tags "Through hole socket strip THT 2x30 2.54mm double row")
-    (property "Sheetfile" "CartdrigeDev.kicad_sch")
+    (property "Sheetfile" "CartdrigeProto.kicad_sch")
     (property "Sheetname" "")
     (property "ki_description" "Generic connector, double row, 02x30, odd/even pin numbering scheme (row 1 odd numbers, row 2 even numbers), script generated (kicad-library-utils/schlib/autogen/connector/)")
