File: Hardware/CartdrigeProto/CartdrigeProto.kicad_sch (KiCad schematic)
At the start: 2 parts, among them J1 Conn_02x30_Odd_Even, J2 PORT1

Commit message: A lot of new hardware
Parts:
- J2: footprint NESConnector:NES_PCBEdge -> Connector_NES:NES_PCBEdge
Changed lines of the file:
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@@
 (kicad_sch (version 20230121) (generator eeschema)
   (paper "A4")
+  (junction (at 30.48 105.41) (diameter 0) (color 0 0 0 0)
+  )
+  (junction (at 30.48 69.85) (diameter 0) (color 0 0 0 0)
+  )
   (no_connect (at 160.02 96.52))
   (no_connect (at 160.02 101.6))
@@
     )
     (property "Datasheet" "~" (at 57.15 67.31 0)
+      (effects (font (size 1.27 1.27)) hide)
+    )
+    (property "Sim.Enable" "0" (at 57.15 67.31 0)
       (effects (font (size 1.27 1.27)) hide)
     )
@@
     (pin "9")
     (instances
-      (project "CartdrigeDev"
+      (project "CartdrigeProto"
         (path "/37e9d49f-81bc-4d5c-bab0-7c054d57d038"
           (reference "J1") (unit 1)
@@
     (pin "1")
     (instances
-      (project "CartdrigeDev"
+      (project "CartdrigeProto"
         (path "/37e9d49f-81bc-4d5c-bab0-7c054d57d038"
           (reference "#PWR02") (unit 1)
@@
     (pin "1")
     (instances
-      (project "CartdrigeDev"
+      (project "CartdrigeProto"
         (path "/37e9d49f-81bc-4d5c-bab0-7c054d57d038"
           (reference "#PWR08") (unit 1)
@@
     )
   )
+  (symbol (lib_id "power:PWR_FLAG") (at 30.48 105.41 180) (unit 1)
+    (in_bom yes) (on_board yes) (dnp no)
+    (property "Reference" "#FLG02" (at 30.48 107.315 0)
+      (effects (font (size 1.27 1.27)) hide)
+    )
+    (property "Value" "PWR_FLAG" (at 25.4 103.505 0)
+      (effects (font (size 1.27 1.27)))
+    )
+    (property "Footprint" "" (at 30.48 105.41 0)
+      (effects (font (size 1.27 1.27)) hide)
+    )
+    (property "Datasheet" "~" (at 30.48 105.41 0)
+      (effects (font (size 1.27 1.27)) hide)
+    )
+    (pin "1")
+    (instances
+      (project "CartdrigeProto"
+        (path "/37e9d49f-81bc-4d5c-bab0-7c054d57d038"
+          (reference "#FLG02") (unit 1)
+        )
+      )
+    )
+  )
   (symbol (lib_id "power:+5V") (at 170.18 26.67 0) (unit 1)
     (in_bom yes) (on_board yes) (dnp no)
@@
     (pin "1")
     (instances
-      (project "CartdrigeDev"
+      (project "CartdrigeProto"
         (path "/37e9d49f-81bc-4d5c-bab0-7c054d57d038"
           (reference "#PWR011") (unit 1)
@@
       (effects (font (size 1.27 1.27)))
     )
-    (property "Footprint" "NESConnector:NES_PCBEdge" (at 152.4 66.04 0)
+    (property "Footprint" "Connector_NES:NES_PCBEdge" (at 152.4 66.04 0)
       (effects (font (size 1.27 1.27)) hide)
     )
     (property "Datasheet" "~" (at 152.4 66.04 0)
+      (effects (font (size 1.27 1.27)) hide)
+    )
+    (property "Sim.Enable" "0" (at 152.4 66.04 0)
       (effects (font (size 1.27 1.27)) hide)
     )
@@
     (pin "9")
     (instances
-      (project "CartdrigeDev"
+      (project "CartdrigeProto"
         (path "/37e9d49f-81bc-4d5c-bab0-7c054d57d038"
           (reference "J2") (unit 1)
@@
     (pin "1")
     (instances
-      (project "CartdrigeDev"
+      (project "CartdrigeProto"
         (path "/37e9d49f-81bc-4d5c-bab0-7c054d57d038"
           (reference "#PWR010") (unit 1)
@@
     (pin "1")
     (instances
-      (project "CartdrigeDev"
+      (project "CartdrigeProto"
         (path "/37e9d49f-81bc-4d5c-bab0-7c054d57d038"
           (reference "#PWR09") (unit 1)
@@
     (pin "1")
     (instances
-      (project "CartdrigeDev"
+      (project "CartdrigeProto"
         (path "/37e9d49f-81bc-4d5c-bab0-7c054d57d038"
           (reference "#PWR04") (unit 1)
@@
     )
   )
+  (symbol (lib_id "power:PWR_FLAG") (at 30.48 69.85 0) (unit 1)
+    (in_bom yes) (on_board yes) (dnp no) (fields_autoplaced)
+    (property "Reference" "#FLG01" (at 30.48 67.945 0)
+      (effects (font (size 1.27 1.27)) hide)
+    )
+    (property "Value" "PWR_FLAG" (at 30.48 64.77 0)
+      (effects (font (size 1.27 1.27)))
+    )
+    (property "Footprint" "" (at 30.48 69.85 0)
+      (effects (font (size 1.27 1.27)) hide)
+    )
+    (property "Datasheet" "~" (at 30.48 69.85 0)
+      (effects (font (size 1.27 1.27)) hide)
+    )
+    (pin "1")
+    (instances
+      (project "CartdrigeProto"
+        (path "/37e9d49f-81bc-4d5c-bab0-7c054d57d038"
+          (reference "#FLG01") (unit 1)
+        )
+      )
+    )
+  )
   (symbol (lib_id "power:+5V") (at 30.48 96.52 0) (unit 1)
     (in_bom yes) (on_board yes) (dnp no)
@@
     (pin "1")
     (instances
-      (project "CartdrigeDev"
+      (project "CartdrigeProto"
         (path "/37e9d49f-81bc-4d5c-bab0-7c054d57d038"
           (reference "#PWR03") (unit 1)
@@
     (pin "1")
     (instances
-      (project "CartdrigeDev"
+      (project "CartdrigeProto"
         (path "/37e9d49f-81bc-4d5c-bab0-7c054d57d038"
           (reference "#PWR01") (unit 1)
