File: Hardware/SerialBoard/SerialBoard.kicad_pcb (KiCad board)
At the start: 2 copper layers, 119.9 x 64.3 mm, 11 parts, among them J1 PORT1, J2 DATA, J3 CTRL, J4 CTRL, J5 DATA, U1 W65C51N, Y1 1.8432MHz

Commit message: Fix
Parts:
- moved J2 24.1 mm to (198.1, 104.1)
- moved J3 24.1 mm to (176.5, 104.1)
- moved J4 24.1 mm to (176.5, 80.0)
- moved J5 24.1 mm to (198.1, 80.0)
Connections:
- J2 pad 1: TX -> RX
- J2 pad 2: RX -> TX
- J3 pad 2: RESET -> unconnected-(J3-Pin_2-Pad2)
- J3 pad 4: DCD -> unconnected-(J3-Pin_4-Pad4)
- J3 pad 5: DSR -> unconnected-(J3-Pin_5-Pad5)
- J3 pad 7: CTS -> unconnected-(J3-Pin_7-Pad7)
- J3 pad 8: RTS -> unconnected-(J3-Pin_8-Pad8)
- U1 pad 16: DCD -> unconnected-(U1-~{DCD}-Pad16)
- U1 pad 17: DSR -> unconnected-(U1-~{DSR}-Pad17)
- U1 pad 8: RTS -> unconnected-(U1-~{RTS}-Pad8)
- U1 pad 9: CTS -> unconnected-(U1-~{CTS}-Pad9)
Routing:
- net DCD: track 77.8 -> 0.00 mm, vias 1 -> 0
- net DSR: track 77.8 -> 0.00 mm, vias 1 -> 0
- net CTS: track 71.6 -> 0.00 mm, vias 1 -> 0
- net RTS: track 69.1 -> 0.00 mm, vias 1 -> 0
- net RESET: track 84.9 -> 43.7 mm, vias 2 -> 1
- net RX: track 95.8 -> 81.8 mm
- net DTR: track 79.3 -> 70.4 mm
- net TX: track 83.1 -> 79.3 mm
